Commit message: fixed1

File: body.urdf (robot description, URDF)
Before this commit: robot robot, 3 links, 2 joints
Joints:
- joint Torso_Backleg: origin xyz=0 -0.5 1 rpy=0 0 0 -> xyz=-0.5 0 1 rpy=0 0 0
- joint Torso_Frontleg: origin xyz=0 -0.5 1 rpy=0 0 0 -> xyz=0.5 0 1 rpy=0 0 0

Commit message: finalN

File: body.urdf (robot description, URDF)
Before this commit: robot robot, 3 links, 2 joints
Links:
- added link Backlowerleg, mass 1; collision box size=0.2 0.2 1; visual box size=0.2 0.2 1
- added link Frontlowerleg, mass 1; collision box size=0.2 0.2 1; visual box size=0.2 0.2 1
- added link Leftleg, mass 1; collision box size=1 0.2 0.2; visual box size=1 0.2 0.2
- added link Leftlowerleg, mass 1; collision box size=0.2 0.2 1; visual box size=0.2 0.2 1
- added link Rightleg, mass 1; collision box size=1 0.2 0.2; visual box size=1 0.2 0.2
- added link Rightlowerleg, mass 1; collision box size=0.2 0.2 1; visual box size=0.2 0.2 1
- link Backleg: geometry collision box size=0.2 1 0.2; visual box size=0.2 1 0.2
- link Frontleg: geometry collision box size=0.2 1 0.2; visual box size=0.2 1 0.2
Joints:
- added joint Backleg_Backlowerleg: type revolute, parent Backleg, child Backlowerleg, origin xyz=0 -1 0 rpy=0 0 0, axis 1 0 0, limit lower=-3.14159 upper=3.14159 effort=0.0 velocity=0.0
- added joint Frontleg_Frontlowerleg: type revolute, parent Frontleg, child Frontlowerleg, origin xyz=0 1 0 rpy=0 0 0, axis 1 0 0, limit lower=-3.14159 upper=3.14159 effort=0.0 velocity=0.0
- added joint Leftleg_Leftlowerleg: type revolute, parent Leftleg, child Leftlowerleg, origin xyz=-1 0 0 rpy=0 0 0, axis 0 1 0, limit lower=-3.14159 upper=3.14159 effort=0.0 velocity=0.0
- added joint Rightleg_Rightlowerleg: type revolute, parent Rightleg, child Rightlowerleg, origin xyz=1 0 0 rpy=0 0 0, axis 0 1 0, limit lower=-3.14159 upper=3.14159 effort=0.0 velocity=0.0
- added joint Torso_Leftleg: type revolute, parent Torso, child Leftleg, origin xyz=-0.5 0 1 rpy=0 0 0, axis 0 1 0, limit lower=-3.14159 upper=3.14159 effort=0.0 velocity=0.0
- added joint Torso_Rightleg: type revolute, parent Torso, child Rightleg, origin xyz=0.5 0 1 rpy=0 0 0, axis 0 1 0, limit lower=-3.14159 upper=3.14159 effort=0.0 velocity=0.0
- joint Torso_Backleg: axis 0 1 0 -> 1 0 0; origin xyz=-0.5 0 1 rpy=0 0 0 -> xyz=0 -0.5 1 rpy=0 0 0
- joint Torso_Frontleg: axis 0 1 0 -> 1 0 0; origin xyz=0.5 0 1 rpy=0 0 0 -> xyz=0 0.5 1 rpy=0 0 0
